File: ProgTan.sch (KiCad schematic (older format))
At the start: 10 parts, among them P1 Power, P2 ESP_A, P3 ESP_B, P4 MOTOR2, P5 MOTOR1, P6 Sensor Proximidad, P7 LM7805, U2 L294D

Commit message: General fixes
Parts:
- added D1, D2: LED, LEDs:LED-3MM, symbol LED
- added P8: Sensor Infrarrojo, Socket_Strips:Socket_Strip_Straight_1x03, symbol CONN_01X03
Connections:
- net GND: now also D1.1 (K), D2.1 (K), P8.3 (P3); no longer P2.2 (P2)
- net GPI00: now also P6.3 (P3)
- net GPI02: now also P6.2 (P2)
- net GPI04: now also P8.2 (P2)
- net GPI12: now also U2.7; no longer P6.2 (P2)
- net GPI14: now also U2.2; no longer P6.3 (P3)
- net Vo: now also P8.1 (P1)
- net GPI10: now reaches P2.3 (P3)
- net GPI10: now also D2.2 (A)
- net GPI09: now reaches P2.4 (P4)
- net GPI09: now also D1.2 (A)
- net GPI01: no longer names the net of P3.13 (P13)
- net GPI01: no longer U2.2
- net GPI03: no longer names the net of P3.12 (P12)
- net GPI03: no longer U2.7
- net GPI05: no longer names the net of P3.2 (P2)
- net GPI16: no longer names the net of P3.1 (P1)
- no-connect marks 13 -> 16
Changed lines of the file:
@@
 Text Label 3840 2800 2    60   ~ 0
 Vo
-Text Label 4790 2590 0    60   ~ 0
-GPI01
-Text Label 4790 2490 0    60   ~ 0
-GPI03
 Text Label 4790 2390 0    60   ~ 0
 GPI15
@@
 Text Label 4790 1590 0    60   ~ 0
 GPI04
-Text Label 4790 1490 0    60   ~ 0
-GPI05
-Text Label 4790 1390 0    60   ~ 0
-GPI16
 $Comp
 L GND #PWR05
@@
 NoConn ~ 3840 2200
 NoConn ~ 3840 1400
-NoConn ~ 3840 1600
-NoConn ~ 3840 1700
 NoConn ~ 3840 1800
 NoConn ~ 3840 1900
@@
 $Comp
 L GND #PWR08
-U 1 1 5AB6AE3F
-P 3645 1500
-F 0 "#PWR08" H 3645 1250 50  0001 C CNN
-F 1 "GND" H 3645 1350 50  0000 C CNN
-F 2 "" H 3645 1500 50  0000 C CNN
-F 3 "" H 3645 1500 50  0000 C CNN
-	1    3645 1500
-	1    0    0    -1
-$EndComp
-$Comp
-L GND #PWR09
 U 1 1 5AB6AE80
 P 3615 2300
-F 0 "#PWR09" H 3615 2050 50  0001 C CNN
+F 0 "#PWR08" H 3615 2050 50  0001 C CNN
 F 1 "GND" H 3615 2150 50  0000 C CNN
 F 2 "" H 3615 2300 50  0000 C CNN
@@
 Wire Wire Line
 	3840 2300 3615 2300
-Wire Wire Line
-	3840 1500 3645 1500
 $Comp
 L IC16 U2
@@
 Vin
 $Comp
-L GND #PWR010
+L GND #PWR09
 U 1 1 5AB6CDBF
 P 6025 1850
-F 0 "#PWR010" H 6025 1600 50  0001 C CNN
+F 0 "#PWR09" H 6025 1600 50  0001 C CNN
 F 1 "GND" H 6025 1700 50  0000 C CNN
 F 2 "" H 6025 1850 50  0000 C CNN
@@
 	7430 1880 7130 1880
 $Comp
-L GND #PWR011
+L GND #PWR010
 U 1 1 5AB6CEBE
 P 7555 1825
-F 0 "#PWR011" H 7555 1575 50  0001 C CNN
+F 0 "#PWR010" H 7555 1575 50  0001 C CNN
 F 1 "GND" H 7555 1675 50  0000 C CNN
 F 2 "" H 7555 1825 50  0000 C CNN
@@
 M2_2
 Text Label 6430 1580 2    60   ~ 0
-GPI01
+GPI14
 Text Label 6430 2080 2    60   ~ 0
-GPI03
+GPI12
 Text Label 7130 1580 0    60   ~ 0
 GPI13
@@
 Vo
 $Comp
-L GND #PWR012
+L GND #PWR011
 U 1 1 5AB6DB17
 P 8750 2645
-F 0 "#PWR012" H 8750 2395 50  0001 C CNN
+F 0 "#PWR011" H 8750 2395 50  0001 C CNN
 F 1 "GND" H 8750 2495 50  0000 C CNN
 F 2 "" H 8750 2645 50  0000 C CNN
@@
 $EndComp
 Text Label 8750 2745 2    60   ~ 0
-GPI12
+GPI02
 Text Label 8750 2845 2    60   ~ 0
-GPI14
+GPI00
 Wire Wire Line
 	2215 1655 2565 1655
@@
 Wire Wire Line
 	2115 1725 2115 1650
-NoConn ~ 4790 1890
 NoConn ~ 4790 2790
 NoConn ~ 3840 2400
@@
 	7940 1030 5830 1030
 Wire Notes Line
-	8235 1025 8235 3440
+	8235 1025 8235 5135
 Wire Notes Line
 	8235 1025 9485 1025
 Wire Notes Line
 	9485 1025 9485 3440
-Wire Notes Line
-	9485 3440 8235 3440
 Text Notes 4050 3145 0    60   ~ 0
 Comunicación
@@
 Text Notes 8355 3365 0    60   ~ 0
 Sensores y actuadores
+NoConn ~ 4790 2590
+NoConn ~ 4790 2490
+$Comp
+L CONN_01X03 P8
+U 1 1 5B05E2F2
+P 8890 3890
+F 0 "P8" H 8890 4090 50  0000 C CNN
+F 1 "Sensor Infrarrojo" V 8990 3890 50  0000 C CNN
+F 2 "Socket_Strips:Socket_Strip_Straight_1x03" H 8890 3890 50  0001 C CNN
+F 3 "" H 8890 3890 50  0000 C CNN
+	1    8890 3890
+	1    0    0    -1
+$EndComp
+Text Label 8690 3790 2    60   ~ 0
+Vo
+Text Label 8690 3890 2    60   ~ 0
+GPI04
+$Comp
+L GND #PWR012
+U 1 1 5B05E5D6
+P 8690 3990
+F 0 "#PWR012" H 8690 3740 50  0001 C CNN
+F 1 "GND" H 8690 3840 50  0000 C CNN
+F 2 "" H 8690 3990 50  0000 C CNN
+F 3 "" H 8690 3990 50  0000 C CNN
+	1    8690 3990
+	1    0    0    -1
+$EndComp
+NoConn ~ 4790 1390
+NoConn ~ 4790 1490
+$Comp
+L LED D1
+U 1 1 5B05EEE9
+P 8610 4630
+F 0 "D1" H 8610 4730 50  0000 C CNN
+F 1 "LED" H 8610 4530 50  0000 C CNN
+F 2 "LEDs:LED-3MM" H 8610 4630 50  0001 C CNN
+F 3 "" H 8610 4630 50  0000 C CNN
+	1    8610 4630
+	0    -1   -1   0
+$EndComp
+$Comp
+L LED D2
+U 1 1 5B05F18A
+P 8945 4630
+F 0 "D2" H 8945 4730 50  0000 C CNN
+F 1 "LED" H 8945 4530 50  0000 C CNN
+F 2 "LEDs:LED-3MM" H 8945 4630 50  0001 C CNN
+F 3 "" H 8945 4630 50  0000 C CNN
+	1    8945 4630
+	0    -1   -1   0
+$EndComp
+$Comp
+L GND #PWR013
+U 1 1 5B05F31C
+P 8775 4885
+F 0 "#PWR013" H 8775 4635 50  0001 C CNN
+F 1 "GND" H 8775 4735 50  0000 C CNN
+F 2 "" H 8775 4885 50  0000 C CNN
+F 3 "" H 8775 4885 50  0000 C CNN
+	1    8775 4885
+	1    0    0    -1
+$EndComp
+Wire Wire Line
+	8610 4830 8945 4830
+Wire Wire Line
+	8775 4885 8775 4830
+Connection ~ 8775 4830
+NoConn ~ 3840 1500
+Text Label 3840 1600 2    60   ~ 0
+GPI10
+Text Label 3840 1700 2    60   ~ 0
+GPI09
+Text Label 8610 4430 2    60   ~ 0
+GPI09
+Text Label 8945 4430 2    60   ~ 0
+GPI10
+NoConn ~ 4790 1890
+Wire Notes Line
+	9485 3430 9485 5135
+Wire Notes Line
+	9485 5135 8235 5135
 $EndSCHEMATC
